File: PCBWay_Version/001.kicad_pcb (KiCad board)
At the start: 2 copper layers, 74.7 x 96.8 mm, 63 parts, among them J1 CONN_01X02, J10 TEST_1P, J11 TEST_1P, J12 TEST_1P, J13 TEST_1P, J14 TEST_1P, J15 TEST_1P, J16 TEST_1P, J2 TEST_1P, J3 TEST_1P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

Commit message: Rev 1
Parts:
- added J17: GS2, Connectors:GS2, B.Cu at (139.6, 96.8)
- added REF***: OSHW-Logo2_7.3x6mm_SilkScreen, Symbols:OSHW-Logo2_7.3x6mm_SilkScreen, B.Cu at (117.8, 57.6)
- C3: value 100uF -> 22nF
- C4: value 10nF -> 22nF
- D1: value DIODE-SCHOTTKY-40V-1A-MBRA140-SMA -> MBRA140; footprint Diodes_SMD:D_SOD-123 -> OSHwi:D_SOD-123
- D2: value RED -> ON; footprint LEDs:LED_1206 -> OSHwi:LED_0805
- GBSilk***, GS***: moved to F.Cu
- J1: footprint Connectors_JST:JST_PH_S2B-PH-SM4-TB_02x2.00mm_Angled -> Connectors_Molex:Molex_PicoBlade_53261-0271_02x1.25mm_Angled
- LED1, LED2, LED3, LED4, LED5: value LED-RGB-WS2812B-4SMD -> WS2812B; footprint Wickerlib:LED-RGB-5050-SMD -> OSHwi:WS2812B
- SW1, SW2: footprint kmr2:SW_SPST_KMR2 -> Buttons_Switches_SMD:SW_SPST_B3U-1000P
- moved R2 3.47 mm to (136.6, 101.7)
- moved GBSilk*** 3.25 mm to (119.0, 106.8), turned to 0 degrees
- moved GS*** 3.25 mm to (119.0, 106.8), turned to 0 degrees
- moved J1 2.65 mm to (130.9, 96.2)
- moved C4 0.68 mm to (134.8, 84.3)
- moved R6 0.50 mm to (118.3, 75.9)
- moved SW2 0.37 mm to (136.7, 101.8)
- moved D2 0.22 mm to (130.9, 101.8)
Connections:
- J9 pad 1: GPIO2 -> GPIO4
- LED1 pad 2: GPIO4 -> GPIO2
- SW1 pad 2: GND -> GPIO0
- SW2 pad 2: GND -> REST
Routing:
- net GPIO12: track 39.1 -> 0.00 mm, vias 3 -> 0
- net CH_PD: track 37.9 -> 51.6 mm, vias 5 -> 3
- net GND: track 9.82 -> 0.00 mm, vias 20 -> 6
- net GPIO16: track 48.6 -> 54.9 mm
- net REST: track 48.1 -> 42.4 mm, vias 1 -> 3
- net GPIO15: track 43.6 -> 38.9 mm, vias 3 -> 1
- net Net-(LED1-Pad4): track 16.7 -> 12.4 mm
- net GPIO13: track 44.0 -> 41.0 mm
- net GPIO5: track 34.9 -> 32.7 mm
- net Net-(D2-Pad2): track 5.68 -> 4.12 mm
- net TXD: track 26.9 -> 25.6 mm
- net RXD: track 32.2 -> 31.2 mm
- net Net-(LED2-Pad4): track 12.5 -> 11.7 mm
- net GPIO4: track 21.9 -> 21.1 mm
- net VCC: track 25.3 -> 24.6 mm
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Other:
- net class Default: trace_width 0.1524 -> 0.25
- net class Power added: clearance 0.1524, trace_width 0.6096, via_dia 0.6858, via_drill 0.3302
- board text added: "+"
- board text added: "-"
- board text added: "4"
- board text added: "DSJ"
- board text added: "RST"
- board text removed: "2"
- board text removed: "REST"

Commit message: REV 1
Parts:
- added G***Ki: Ki-LOGO, varios:Ki-2500, B.Cu at (142.1, 57.6)
- added G***TME: LOGO-TME, varios:TME-1500, B.Cu at (118.7, 106.9)
- GBSilk***, GS***: moved to B.Cu
- moved GBSilk*** 5.69 mm to (122.3, 102.2), turned to 180 degrees
- moved GS*** 5.69 mm to (122.3, 102.2), turned to 180 degrees
- moved R6 0.98 mm to (118.8, 76.7)
Routing:
- net GPIO12: track 0.00 -> 40.1 mm, vias 0 -> 2
- net GPIO4: track 21.1 -> 32.9 mm, vias 1 -> 4
- net CH_PD: track 51.6 -> 40.0 mm
- net GPIO15: track 38.9 -> 45.0 mm
- net REST: track 42.4 -> 47.1 mm
- net GND: track 0.00 -> 3.86 mm, vias 6 -> 17
- net GPIO13: track 41.0 -> 37.9 mm
- net GPIO16: track 54.9 -> 53.3 mm
- net GPIO2: track 37.4 -> 38.7 mm, vias 2 -> 1
- net +3.3V: track 160.9 -> 161.8 mm
- net GPIO14: track 42.6 -> 43.5 mm
- net GPIO0: track 50.1 -> 50.8 mm
- net RXD: track 31.2 -> 31.8 mm
- net GPIO5: track 32.7 -> 33.2 mm
