File: PCBWay_Version/001.sch (KiCad schematic (older format))
At the start: 38 parts, among them J1 CONN_01X02, J10 TEST_1P, J11 TEST_1P, J12 TEST_1P, J13 TEST_1P, J14 TEST_1P, J15 TEST_1P, J16 TEST_1P, J2 TEST_1P, J3 TEST_1P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

Commit message: Rev 1
Parts:
- removed C3: 100uF, Capacitors_SMD:C_0805_HandSoldering, symbol CP
- added C3: 22nF, Capacitors_SMD:C_0805_HandSoldering, symbol CAP
- added J17: GS2, Connectors:GS2, symbol GS2
- C4: value 10nF -> 22nF
- D1: value DIODE-SCHOTTKY-40V-1A-MBRA140-SMA -> MBRA140; footprint Diodes_SMD:D_SOD-123 -> OSHwi:D_SOD-123
- D2: value RED -> ON; footprint LEDs:LED_1206 -> OSHwi:LED_0805
- J1: footprint Connectors_JST:JST_PH_S2B-PH-SM4-TB_02x2.00mm_Angled -> Connectors_Molex:Molex_PicoBlade_53261-0271_02x1.25mm_Angled
- LED1, LED2, LED3, LED4, LED5: value LED-RGB-WS2812B-4SMD -> WS2812B; footprint Wickerlib:LED-RGB-5050-SMD -> OSHwi:WS2812B
- SW1, SW2: footprint kmr2:SW_SPST_KMR2 -> Buttons_Switches_SMD:SW_SPST_B3U-1000P; symbol SWITCH-MOMENT-SPDT-SMT-B3FS-4002P -> SW_Push
Connections:
- net +3.3V: now also C3.1
- net GND: now also C3.2; no longer SW1.2, SW2.2
- net GPIO0: now also SW1.2; no longer SW1.3, SW1.4
- net GPIO16: now also J17.2 (G2)
- net GPIO2: now also LED1.2 (DI); no longer J9.1
- net GPIO4: now also J9.1; no longer LED1.2 (DI)
- net REST: now also SW2.2, J17.1 (G1); no longer SW2.3, SW2.4
Other:
- note added: "DEEP SLEEP"
- moved on the sheet: D2, R1, R2, R3, R4, R6, R7
