File: Oshpark_Version/001.sch (KiCad schematic (older format))
At the start: 39 parts, among them J1 CONN_01X02, J10 TEST_1P, J11 TEST_1P, J12 TEST_1P, J13 TEST_1P, J14 TEST_1P, J15 TEST_1P, J16 TEST_1P, J17 GS2, J2 TEST_1P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

Commit message: Add Schematic PDF
Parts:
- U2: symbol SPX3819M5-L-1-8 -> SPX3819M5-L-1-8-RESCUE-001
Changed lines of the file:
@@
 EESchema Schematic File Version 2
+LIBS:001-rescue
 LIBS:bbd
 LIBS:battery_management
@@
 LIBS:kmr2
 LIBS:001-cache
-EELAYER 26 0
+EELAYER 25 0
 EELAYER END
 $Descr USLetter 11000 8500
@@
 VBAT
 $Comp
-L SPX3819M5-L-1-8 U2
+L SPX3819M5-L-1-8-RESCUE-001 U2
 U 1 1 5980EF98
 P 8150 1275
