File: Hackster_Version/001.kicad_pcb (KiCad board)
At the start: 2 copper layers, 74.7 x 96.8 mm, 75 parts, among them J1 CONN_01X02, J10 TEST_1P, J11 TEST_1P, J12 TEST_1P, J13 TEST_1P, J14 TEST_1P, J15 TEST_1P, J16 TEST_1P, J17 GS2, J2 TEST_1P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

Commit message: Auto stash before merge of "master" and "origin/master"
Routing:
- net GPIO4: track 32.9 -> 36.9 mm
- net Net-(LED4-Pad4): track 13.3 -> 15.6 mm
- net REST: track 47.1 -> 49.0 mm
- net GPIO16: track 53.3 -> 54.8 mm
- net GPIO12: track 40.1 -> 39.2 mm
- net +3.3V: track 161.8 -> 162.6 mm
- net GPIO13: track 37.9 -> 37.1 mm
- net ADC: track 41.7 -> 41.0 mm
- net GPIO15: track 45.0 -> 45.6 mm
- net TXD: track 25.6 -> 25.1 mm
- net GND: track 3.86 -> 3.65 mm, vias 17 -> 22
