File: Hackster_Version/001.sch (KiCad schematic (older format))
At the start: 39 parts, among them J1 CONN_01X02, J10 TEST_1P, J11 TEST_1P, J12 TEST_1P, J13 TEST_1P, J14 TEST_1P, J15 TEST_1P, J16 TEST_1P, J17 GS2, J2 TEST_1P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

Commit message: Update Buttom Reset description
Parts:
- removed SW2: RESET, Buttons_Switches_SMD:SW_SPST_B3U-1000P, symbol SW_Push
- added SW2: RESET, Buttons_Switches_SMD:SW_SPST_B3U-1000P, symbol switches:SW_Push
- C1, C2, C3, C4: symbol CAP -> pspice:CAP
- D1: symbol DIODE-SCHOTTKY-40V-1A-MBRA140-SMA -> wickerlib:DIODE-SCHOTTKY-40V-1A-MBRA140-SMA
- D2: symbol LED -> device:LED
- J1: symbol CONN_01X02 -> conn:CONN_01X02
- J10, J11, J12, J13, J14, J15, J16, J2, J3, J4, J5, J6, J7, J8, J9: symbol TEST_1P -> conn:TEST_1P
- J17: symbol GS2 -> conn:GS2
- LED1, LED2, LED3, LED4, LED5: symbol LED-RGB-WS2812B-4SMD -> wickerlib:LED-RGB-WS2812B-4SMD
- R1, R2, R3, R4, R5, R6, R7: symbol R -> pspice:R
- SW1: symbol SW_Push -> switches:SW_Push; Description SWITCH MOMENT SPST-NO 0.05A 24V SMT B3FS-4002P -> B3U-1000P - Tactile Switch, Ultra Small, Non Illuminated, 1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
- U1: symbol ESP-12 -> ESP8266:ESP-12
- U2: symbol SPX3819M5-L-1-8-RESCUE-001 -> 001-rescue:SPX3819M5-L-1-8-RESCUE-001
Connections:
- wire segments 70 -> 84
