File: 2019/Oshwi_M0/_autosave-001.sch (KiCad schematic (older format))
At the start: 71 parts, among them CN1 MICROSD, IC1 APX803, J1 Conn_01x01, J10 Conn_01x01, J11 Conn_01x01, J12 Conn_01x01, J2 Conn_01x01, J3 Conn_01x01, J4 Conn_01x01, J5 Conn_01x01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

Commit message: Add Schematic for TFT & PyPortal
Parts:
- removed JP2: HEADER-1X16ROUND, Oshwi_M0:1X16_ROUND, symbol 001-rescue:HEADER-1X16ROUND-Adafruit_Feather_M0_Express-eagle-import
- CHG1, L1: symbol Device:LED -> 001-rescue:LED-Device
- J1, J10, J11, J12, J2, J3, J4, J5, J6, J7, J8, J9, J? (x16): symbol Connector:Conn_01x01_Female -> 001-rescue:Conn_01x01_Female-Connector
- SW1: symbol Switch:SW_Push -> 001-rescue:SW_Push-Switch
Connections:
- wire segments 219 -> 217
Changed lines of the file:
@@
 	10250 5275 10250 5375
-Wire Wire Line
-	9800 6475 10200 6475
-Wire Wire Line
-	10400 6600 10400 6700
 Wire Wire Line
 	3450 2275 3450 1975
@@
 	1    6350 4175
 	0    -1   -1   0
-$EndComp
-$Comp
-L 001-rescue:HEADER-1X16ROUND-Adafruit_Feather_M0_Express-eagle-import JP2
-U 1 1 5CCCC11E
-P 9125 7275
-F 0 "JP2" H 8875 8100 59  0000 L BNN
-F 1 "HEADER-1X16ROUND" H 8875 6275 59  0000 L BNN
-F 2 "Oshwi_M0:1X16_ROUND" H 9125 7275 50  0001 C CNN
-F 3 "" H 9125 7275 50  0001 C CNN
-	1    9125 7275
-	-1   0    0    1
 $EndComp
 $Comp
@@
 Connection ~ 1000 4200
 $Comp
-L Device:LED CHG1
+L 001-rescue:LED-Device CHG1
 U 1 1 5CCC697A
 P 6150 1525
@@
 $EndComp
 $Comp
-L Device:LED L1
+L 001-rescue:LED-Device L1
 U 1 1 5CCCC16E
 P 10250 5125
@@
 $EndComp
 $Comp
-L Switch:SW_Push SW1
+L 001-rescue:SW_Push-Switch SW1
 U 1 1 5CC54900
 P 5450 1375
@@
 $EndComp
 $Comp
-L Connector:Conn_01x01_Female J1
+L 001-rescue:Conn_01x01_Female-Connector J1
 U 1 1 5CC4E09B
 P 7350 4175
@@
 $EndComp
 $Comp
-L Connector:Conn_01x01_Female J2
+L 001-rescue:Conn_01x01_Female-Connector J2
 U 1 1 5CC50EE1
 P 7350 4275
@@
 $EndComp
 $Comp
-L Connector:Conn_01x01_Female J3
+L 001-rescue:Conn_01x01_Female-Connector J3
 U 1 1 5CC51194
 P 7350 4375
@@
 $EndComp
 $Comp
-L Connector:Conn_01x01_Female J4
+L 001-rescue:Conn_01x01_Female-Connector J4
 U 1 1 5CC5239F
 P 7350 4475
@@
 $EndComp
 $Comp
-L Connector:Conn_01x01_Female J5
+L 001-rescue:Conn_01x01_Female-Connector J5
 U 1 1 5CC523AA
 P 7350 4575
@@
 $EndComp
 $Comp
-L Connector:Conn_01x01_Female J6
+L 001-rescue:Conn_01x01_Female-Connector J6
 U 1 1 5CC523B5
 P 7350 4675
@@
 $EndComp
 $Comp
-L Connector:Conn_01x01_Female J7
+L 001-rescue:Conn_01x01_Female-Connector J7
 U 1 1 5CC54BD1
 P 7350 4775
@@
 $EndComp
 $Comp
-L Connector:Conn_01x01_Female J8
+L 001-rescue:Conn_01x01_Female-Connector J8
 U 1 1 5CC54BDC
 P 7350 4875
@@
 $EndComp
 $Comp
-L Connector:Conn_01x01_Female J9
+L 001-rescue:Conn_01x01_Female-Connector J9
 U 1 1 5CC54BE7
 P 7350 4975
@@
 $EndComp
 $Comp
-L Connector:Conn_01x01_Female J10
+L 001-rescue:Conn_01x01_Female-Connector J10
 U 1 1 5CC54BF2
 P 7350 5075
@@
 $EndComp
 $Comp
-L Connector:Conn_01x01_Female J11
+L 001-rescue:Conn_01x01_Female-Connector J11
 U 1 1 5CC54BFD
 P 7350 5175
@@
 $EndComp
 $Comp
-L Connector:Conn_01x01_Female J12
+L 001-rescue:Conn_01x01_Female-Connector J12
 U 1 1 5CC54C08
 P 7350 5275
@@
 $EndComp
 $Comp
-L Connector:Conn_01x01_Female J?
+L 001-rescue:Conn_01x01_Female-Connector J?
 U 1 1 5CC5B3C7
 P 9150 4175
@@
 $EndComp
 $Comp
-L Connector:Conn_01x01_Female J?
+L 001-rescue:Conn_01x01_Female-Connector J?
 U 1 1 5CC5B3D2
 P 9150 4275
@@
 $EndComp
 $Comp
-L Connector:Conn_01x01_Female J?
+L 001-rescue:Conn_01x01_Female-Connector J?
 U 1 1 5CC5B3DD
 P 9150 4400
@@
 $EndComp
 $Comp
-L Connector:Conn_01x01_Female J?
+L 001-rescue:Conn_01x01_Female-Connector J?
 U 1 1 5CC5B3F3
 P 9150 4600
@@
 $EndComp
 $Comp
-L Connector:Conn_01x01_Female J?
+L 001-rescue:Conn_01x01_Female-Connector J?
 U 1 1 5CC5B3FE
 P 9150 4700
@@
 $EndComp
 $Comp
-L Connector:Conn_01x01_Female J?
+L 001-rescue:Conn_01x01_Female-Connector J?
 U 1 1 5CC5B409
 P 9150 4800
@@
 $EndComp
 $Comp
-L Connector:Conn_01x01_Female J?
+L 001-rescue:Conn_01x01_Female-Connector J?
 U 1 1 5CC5B414
 P 9150 4900
@@
 $EndComp
 $Comp
-L Connector:Conn_01x01_Female J?
+L 001-rescue:Conn_01x01_Female-Connector J?
 U 1 1 5CC5B41F
 P 9150 5000
@@
 $EndComp
 $Comp
-L Connector:Conn_01x01_Female J?
+L 001-rescue:Conn_01x01_Female-Connector J?
 U 1 1 5CC5B42A
 P 9150 5100
@@
 $EndComp
 $Comp
-L Connector:Conn_01x01_Female J?
+L 001-rescue:Conn_01x01_Female-Connector J?
 U 1 1 5CC5B435
 P 9150 5200
@@
 $EndComp
 $Comp
-L Connector:Conn_01x01_Female J?
+L 001-rescue:Conn_01x01_Female-Connector J?
 U 1 1 5CC5B440
 P 9150 5300
@@
 $EndComp
 $Comp
-L Connector:Conn_01x01_Female J?
+L 001-rescue:Conn_01x01_Female-Connector J?
 U 1 1 5CC62A14
 P 9150 5400
@@
 $EndComp
 $Comp
-L Connector:Conn_01x01_Female J?
+L 001-rescue:Conn_01x01_Female-Connector J?
 U 1 1 5CC62A1F
 P 9150 5500
@@
 $EndComp
 $Comp
-L Connector:Conn_01x01_Female J?
+L 001-rescue:Conn_01x01_Female-Connector J?
 U 1 1 5CC62A2A
 P 9150 5600
@@
 $EndComp
 $Comp
-L Connector:Conn_01x01_Female J?
+L 001-rescue:Conn_01x01_Female-Connector J?
 U 1 1 5CC64120
 P 9150 5700
@@
 	8350 4400 8950 4400
 $Comp
-L Connector:Conn_01x01_Female J?
+L 001-rescue:Conn_01x01_Female-Connector J?
 U 1 1 5CC71CF1
 P 9150 4500
