File: 2019/Oshwi_M0/001.sch (KiCad schematic (older format))
At the start: 69 parts, among them CN1 MICROSD, IC1 APX803, J1 Conn_01x01, J10 Conn_01x01, J11 Conn_01x01, J12 Conn_01x01, J13 Conn_01x01, J14 Conn_01x01, J15 Conn_01x01, J16 Conn_01x01, J17 Conn_01x01, J18 Conn_01x01, J19 Conn_01x01, J2 Conn_01x01, J20 Conn_01x01, J21 Conn_01x01, J22 Conn_01x01, J23 Conn_01x01, J24 Conn_01x01, J25 Conn_01x01, J26 Conn_01x01, J27 Conn_01x01, J28 Conn_01x01, J3 Conn_01x01, J4 Conn_01x01, J5 Conn_01x01, J6 Conn_01x01, J7 Conn_01x01, J8 Conn_01x01, J9 Conn_01x01, Q1 MMBT2222, SW1 SW_Push, U1 AP2112-3.3, U2 MCP73831T-2ACI/OT, U3 2MB Flash, X1 JSTPH, X2 32.768, X3 microUSB

Commit message: Updates
Parts:
- added LED2, LED3, LED4, LED5: WS2812B3535, OSHwi:WS2812B, symbol 001-rescue:WS2812B3535-Adafruit_Feather_M0_Express-eagle-import
Connections:
- wire segments 201 -> 226
Other:
- note added: "MICRO SD"
- moved on the sheet: C11, CN1, IC1, J1, J10, J11, J12, J13, J14, J15, J16, J17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

Commit message: updates
Parts:
- renumbered C2 to C1, C11 to C10, C1 to C2, JP3 to JP1
Connections:
- wire segments 226 -> 231

Commit message: Remove Bad commits & Update SPI Symbol
Parts:
- removed C9: 10µF, OSHwi:C_0805_HandSoldering, symbol 001-rescue:CAP_CERAMIC0805-NOOUTLINE-Adafruit_Feather_M0_Express-eagle-import
- removed CHG1: ORANGE, OSHwi:LED_0805, symbol 001-rescue:LED-Device
- removed J1, J13, J15, J2, J3: Conn_01x01, OSHwi:CONN-HEADER-STRAIGHT-P2.54MM-1x01, symbol 001-rescue:Conn_01x01_Female-Connector
- removed R3: 1K, OSHwi:R_0805_HandSoldering, symbol 001-rescue:RESISTOR_0603_NOOUT-Adafruit_Feather_M0_Express-eagle-import
- removed R4: 10K, OSHwi:R_0805_HandSoldering, symbol 001-rescue:RESISTOR_0603_NOOUT-Adafruit_Feather_M0_Express-eagle-import
- removed U2: MCP73831T-2ACI/OT, OSHwi:SOT-23-5_HandSoldering, symbol 001-rescue:MCP73831_2-Adafruit_Feather_M0_Express-eagle-import
- removed U3: 2MB Flash, Oshwi_M0:SOIC8_208MIL, symbol 001-rescue:SPIFLASH_SOIC8208MIL-Adafruit_Feather_M0_Express-eagle-import
- added U2: SPIFLASH_SOIC8208MIL, symbol 001-rescue:SPIFLASH_SOIC8208MIL-Adafruit_Feather_M0_Express-eagle-import
- renumbered C5 to C2, C6 to C3, C2 to C4, C3 to C5, C4 to C6, C1 to C9, J4 to J1, J18 to J10, J10 to J11, J19 to J12, J11 to J13, J20 to J14, J12 to J15, J21 to J16, J22 to J17, J23 to J18, J24 to J19, J5 to J2, J25 to J20, J26 to J21, J27 to J22, J28 to J23, J14 to J3, J6 to J4, J7 to J5, J16 to J6, J8 to J7, J17 to J8, R6 to R1, R9 to R10, R5 to R11, R7 to R2, R1 to R3, R2 to R6, R10 to R7, R11 to R9, U$1 to U4, U$2 to U5, X3 to X1, X1 to X2, X2 to X3
Connections:
- net labels removed: EN
- wire segments 231 -> 208
Other:
- note added: "USB"
- note removed: "1.0K = 1000mA"
- note removed: "10K = 100mA"
- note removed: "2.0K = 500mA"
- note removed: "5.0K = 200mA"
- note removed: "USB AND BATTERY CHARGING"
- moved on the sheet: J1, J10, J11, J12, J13, J14, J15, J16, J17, J18, J19, J2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

Commit message: Update SAMD21G Symbol & add CE schematic
Parts:
- removed C7, C8: 22pF, OSHwi:C_0805_HandSoldering, symbol 001-rescue:CAP_CERAMIC0603_NO-Adafruit_Feather_M0_Express-eagle-import
- removed C9: 1uF, OSHwi:C_0805_HandSoldering, symbol 001-rescue:CAP_CERAMIC0603_NO-Adafruit_Feather_M0_Express-eagle-import
- removed TP1, TP2: TESTPOINTROUND1.5MM, Oshwi_M0:TESTPOINT_ROUND_1.5MM, symbol 001-rescue:TESTPOINTROUND1.5MM-Adafruit_Feather_M0_Express-eagle-import
- removed U4: ATSAMD21G18_QFN, Oshwi_M0:TQFN48_7MM, symbol 001-rescue:ATSAMD21G_QFN-Adafruit_Feather_M0_Express-eagle-import
- removed X3: 32.768, Oshwi_M0:XTAL3215, symbol 001-rescue:XTAL-3.2X1.5-Adafruit_Feather_M0_Express-eagle-import
- added 3.3VTAP?, 3V3TAP?, D?, GND3TAP?, GNDTAP? (x2), IO? (x3), RX?, SCL?, SDA?, TX?, VCC?: SEWTAP-ALLIGATOR, Adafruit Circuit Playground Express:SEWALLI, symbol Adafruit_Circuit_Playground_Express-eagle-import:SEWTAP-ALLIGATOR
- added BATT?: 3-6VDC, Adafruit Circuit Playground Express:JSTPH2, symbol Adafruit_Circuit_Playground_Express-eagle-import:CON_JST_PH_2PIN
- added C1: 1uF, symbol device:C_Small
- added C7, C9: 22pF, symbol device:C_Small
- added C? (x5): 1uF, Adafruit Circuit Playground Express:0603-NO, symbol Adafruit_Circuit_Playground_Express-eagle-import:CAP_CERAMIC0603_NO
- added C? (x2): 10uF, Adafruit Circuit Playground Express:0805-NO, symbol Adafruit_Circuit_Playground_Express-eagle-import:CAP_CERAMIC0805-NOOUTLINE
- added CN?: MicroB USB, Adafruit Circuit Playground Express:4UCONN_20329_V2, symbol Adafruit_Circuit_Playground_Express-eagle-import:USB_MICRO_20329_V2
- added D?: IR TX, Adafruit Circuit Playground Express:CHIPLED_1206_NOOUTLINE, symbol Adafruit_Circuit_Playground_Express-eagle-import:LED1206_NOOUTLINE
- added D? (x2): MBR120, Adafruit Circuit Playground Express:SOD-123, symbol Adafruit_Circuit_Playground_Express-eagle-import:DIODESOD-123
- added F?: 6V+ 500mA, Adafruit Circuit Playground Express:R1206, symbol Adafruit_Circuit_Playground_Express-eagle-import:PTCFUSE-1206
- added J24, J25: TEST_1P, symbol conn:TEST_1P
- added J?: Micro_SD_Card_Det, symbol conn:Micro_SD_Card_Det
- added L?: RED, Adafruit Circuit Playground Express:CHIPLED_0805_NOOUTLINE, symbol Adafruit_Circuit_Playground_Express-eagle-import:LED0805_NOOUTLINE
- added LED? (x6): WS2812B3535, Adafruit Circuit Playground Express:LED3535, symbol Adafruit_Circuit_Playground_Express-eagle-import:WS2812B3535
- added PWR?: GREEN, Adafruit Circuit Playground Express:CHIPLED_0805_NOOUTLINE, symbol Adafruit_Circuit_Playground_Express-eagle-import:LED0805_NOOUTLINE
- added Q?: mmbt2222, Adafruit Circuit Playground Express:SOT23-R, symbol Adafruit_Circuit_Playground_Express-eagle-import:TRANSISTOR_NPN
- added R? (x2): 1K, Adafruit Circuit Playground Express:0603-NO, symbol Adafruit_Circuit_Playground_Express-eagle-import:RESISTOR_0603_NOOUT
- added R?: 100, Adafruit Circuit Playground Express:0603-NO, symbol Adafruit_Circuit_Playground_Express-eagle-import:RESISTOR_0603_NOOUT
- added R? (x2): 10k, Adafruit Circuit Playground Express:0603-NO, symbol Adafruit_Circuit_Playground_Express-eagle-import:RESISTOR_0603_NOOUT
- added RESET?: KMR2, Adafruit Circuit Playground Express:BTN_KMR2_4.6X2.8, symbol Adafruit_Circuit_Playground_Express-eagle-import:SWITCH_TACT_SMT4.6X2.8
- added SW? (x2): EVQQ, Adafruit Circuit Playground Express:EVQ-Q2_SMALLER, symbol Adafruit_Circuit_Playground_Express-eagle-import:SWITCH_TACT_SMT_EVQQ2_SMALL
- added SWITCH? (x2): EG1390, Adafruit Circuit Playground Express:EG1390, symbol Adafruit_Circuit_Playground_Express-eagle-import:DPDT-EG1390
- added TP? (x2): TESTPOINTROUND1.5MM, Adafruit Circuit Playground Express:TESTPOINT_ROUND_1.5MM, symbol Adafruit_Circuit_Playground_Express-eagle-import:TESTPOINTROUND1.5MM
- added U$?: ATSAMD21G18MU, Adafruit Circuit Playground Express:TQFN48_7MM, symbol Adafruit_Circuit_Playground_Express-eagle-import:ATSAMD21G_QFN
- added U3: ATSAMD21G18A-AUT, Package_QFP:TQFP-48_7x7mm_P0.5mm, symbol oshwi_M0:ATSAMD21G18A-AUT
- added U?: SPI FLASH, Adafruit Circuit Playground Express:SOIC8_150MIL, symbol Adafruit_Circuit_Playground_Express-eagle-import:SPIFLASH_SOIC8
- added U?: AP2112K-3.3, Adafruit Circuit Playground Express:SOT23-5, symbol Adafruit_Circuit_Playground_Express-eagle-import:VREG_SOT23-5
- added Y1: 32.768, symbol device:Crystal
Connections:
- net labels added: 1.2V, 3.3V, A8_LIGHT, A9_TEMP_SENSE, D0_A6_RX, D10_A3, D12_A0_SPEAKER, D13_LED, D1_A7_TX, D29_REMOTEOUT, D2_A5_SDA, D2_FLASH_MISO, D32_FLASH_MISO, D33_FLASH_SCK, D34_FLASH_MOSI, D35_FLASH_CS, D36_LISIRQ, D3_A4_SCL, D3_FLASH_SCK, D4_FLASH_MOSI, D4_LEFTBUTTON, D5_RIGHTBUTTON, D6_A1, D7_SLIDESWITCH, D9_A2, I2S_DO, I2S_SCK, IR_ANALOGIN, LIS_SCL, LIS_SDA, REMOTEIN, SWCLK/SPK_SD, VCC
- wire segments 208 -> 335
- no-connect marks 10 -> 11
Other:
- note added: "3.3V Reg"
- note added: "ATSAMD21 MICROCONTROLLER"
- note added: "Capacitive Touch/IO Pads"
- note added: "JST Battery In"
- note added: "LEDs"
- note added: "NeoPixels"
- note added: "POWER SUPPLY"
- note added: "SERCOM 1: internal I2C\nSERCOM 3: internal SPI\nSERCOM 4: Serial\nSERCOM 5: external I2C"
- note added: "SPI FLASH"
- note added: "Slide Switch"
- note added: "TXLED"
- note added: "Tact Switch"
- note added: "USB Power/Data"
- note added: "Y0"
- note added: "Y1"
- note added: "Y14"
- note added: "Y15"
- note added: "Y2"
- note added: "Y3"
- note added: "Y4"
- note added: "Y5"
- note added: "Y8"
- note added: "Y9"
- moved on the sheet: C10, C2, C3, C4, C5, C6, CN1, D1, IC1, J1, J10, J11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

Commit message: Add CE Symbol
Parts:
- removed C?: 1uF, Adafruit Circuit Playground Express:0603-NO, symbol Adafruit_Circuit_Playground_Express-eagle-import:CAP_CERAMIC0603_NO
- 3.3VTAP1: renamed from 3.3VTAP?; symbol Adafruit_Circuit_Playground_Express-eagle-import:SEWTAP-ALLIGATOR -> 001-rescue:SEWTAP-ALLIGATOR-Adafruit_Circuit_Playground_Express-eagle-import
- 3V3TAP1: renamed from 3V3TAP?; symbol Adafruit_Circuit_Playground_Express-eagle-import:SEWTAP-ALLIGATOR -> 001-rescue:SEWTAP-ALLIGATOR-Adafruit_Circuit_Playground_Express-eagle-import
- BATT1: renamed from BATT?; symbol Adafruit_Circuit_Playground_Express-eagle-import:CON_JST_PH_2PIN -> 001-rescue:CON_JST_PH_2PIN-Adafruit_Circuit_Playground_Express-eagle-import
- C11, C13, C14, C15: renamed from C?; symbol Adafruit_Circuit_Playground_Express-eagle-import:CAP_CERAMIC0603_NO -> 001-rescue:CAP_CERAMIC0603_NO-Adafruit_Circuit_Playground_Express-eagle-import
- C12, C8: renamed from C?; symbol Adafruit_Circuit_Playground_Express-eagle-import:CAP_CERAMIC0805-NOOUTLINE -> 001-rescue:CAP_CERAMIC0805-NOOUTLINE-Adafruit_Circuit_Playground_Express-eagle-import
- CN2: renamed from CN?; symbol Adafruit_Circuit_Playground_Express-eagle-import:USB_MICRO_20329_V2 -> 001-rescue:USB_MICRO_20329_V2-Adafruit_Circuit_Playground_Express-eagle-import
- D2: renamed from D?; symbol Adafruit_Circuit_Playground_Express-eagle-import:SEWTAP-ALLIGATOR -> 001-rescue:SEWTAP-ALLIGATOR-Adafruit_Circuit_Playground_Express-eagle-import
- D3: renamed from D?; symbol Adafruit_Circuit_Playground_Express-eagle-import:LED1206_NOOUTLINE -> 001-rescue:LED1206_NOOUTLINE-Adafruit_Circuit_Playground_Express-eagle-import
- D4, D5: renamed from D?; symbol Adafruit_Circuit_Playground_Express-eagle-import:DIODESOD-123 -> 001-rescue:DIODESOD-123-Adafruit_Circuit_Playground_Express-eagle-import
- F1: renamed from F?; symbol Adafruit_Circuit_Playground_Express-eagle-import:PTCFUSE-1206 -> 001-rescue:PTCFUSE-1206-Adafruit_Circuit_Playground_Express-eagle-import
- GND3TAP1: renamed from GND3TAP?; symbol Adafruit_Circuit_Playground_Express-eagle-import:SEWTAP-ALLIGATOR -> 001-rescue:SEWTAP-ALLIGATOR-Adafruit_Circuit_Playground_Express-eagle-import
- GNDTAP1, GNDTAP2: renamed from GNDTAP?; symbol Adafruit_Circuit_Playground_Express-eagle-import:SEWTAP-ALLIGATOR -> 001-rescue:SEWTAP-ALLIGATOR-Adafruit_Circuit_Playground_Express-eagle-import
- IO1, IO2, IO3: renamed from IO?; symbol Adafruit_Circuit_Playground_Express-eagle-import:SEWTAP-ALLIGATOR -> 001-rescue:SEWTAP-ALLIGATOR-Adafruit_Circuit_Playground_Express-eagle-import
- L2: renamed from L?; symbol Adafruit_Circuit_Playground_Express-eagle-import:LED0805_NOOUTLINE -> 001-rescue:LED0805_NOOUTLINE-Adafruit_Circuit_Playground_Express-eagle-import
- LED10, LED11, LED6, LED7, LED8, LED9: renamed from LED?; symbol Adafruit_Circuit_Playground_Express-eagle-import:WS2812B3535 -> 001-rescue:WS2812B3535-Adafruit_Circuit_Playground_Express-eagle-import
- PWR1: renamed from PWR?; symbol Adafruit_Circuit_Playground_Express-eagle-import:LED0805_NOOUTLINE -> 001-rescue:LED0805_NOOUTLINE-Adafruit_Circuit_Playground_Express-eagle-import
- Q2: renamed from Q?; symbol Adafruit_Circuit_Playground_Express-eagle-import:TRANSISTOR_NPN -> 001-rescue:TRANSISTOR_NPN-Adafruit_Circuit_Playground_Express-eagle-import
- R12, R13, R14, R4, R5: renamed from R?; symbol Adafruit_Circuit_Playground_Express-eagle-import:RESISTOR_0603_NOOUT -> 001-rescue:RESISTOR_0603_NOOUT-Adafruit_Circuit_Playground_Express-eagle-import
- RESET1: renamed from RESET?; symbol Adafruit_Circuit_Playground_Express-eagle-import:SWITCH_TACT_SMT4.6X2.8 -> 001-rescue:SWITCH_TACT_SMT4.6X2.8-Adafruit_Circuit_Playground_Express-eagle-import
- RX1: renamed from RX?; symbol Adafruit_Circuit_Playground_Express-eagle-import:SEWTAP-ALLIGATOR -> 001-rescue:SEWTAP-ALLIGATOR-Adafruit_Circuit_Playground_Express-eagle-import
- SCL1: renamed from SCL?; symbol Adafruit_Circuit_Playground_Express-eagle-import:SEWTAP-ALLIGATOR -> 001-rescue:SEWTAP-ALLIGATOR-Adafruit_Circuit_Playground_Express-eagle-import
- SDA1: renamed from SDA?; symbol Adafruit_Circuit_Playground_Express-eagle-import:SEWTAP-ALLIGATOR -> 001-rescue:SEWTAP-ALLIGATOR-Adafruit_Circuit_Playground_Express-eagle-import
- SW2, SW3: renamed from SW?; symbol Adafruit_Circuit_Playground_Express-eagle-import:SWITCH_TACT_SMT_EVQQ2_SMALL -> 001-rescue:SWITCH_TACT_SMT_EVQQ2_SMALL-Adafruit_Circuit_Playground_Express-eagle-import
- SWITCH1: renamed from SWITCH?; symbol Adafruit_Circuit_Playground_Express-eagle-import:DPDT-EG1390 -> 001-rescue:DPDT-EG1390-Adafruit_Circuit_Playground_Express-eagle-import
- TP1, TP2: renamed from TP?; symbol Adafruit_Circuit_Playground_Express-eagle-import:TESTPOINTROUND1.5MM -> 001-rescue:TESTPOINTROUND1.5MM-Adafruit_Circuit_Playground_Express-eagle-import
- TX1: renamed from TX?; symbol Adafruit_Circuit_Playground_Express-eagle-import:SEWTAP-ALLIGATOR -> 001-rescue:SEWTAP-ALLIGATOR-Adafruit_Circuit_Playground_Express-eagle-import
- U$1: renamed from U$?; symbol Adafruit_Circuit_Playground_Express-eagle-import:ATSAMD21G_QFN -> 001-rescue:ATSAMD21G_QFN-Adafruit_Circuit_Playground_Express-eagle-import
- U4: renamed from U?; symbol Adafruit_Circuit_Playground_Express-eagle-import:SPIFLASH_SOIC8 -> 001-rescue:SPIFLASH_SOIC8-Adafruit_Circuit_Playground_Express-eagle-import
- U6: renamed from U?; symbol Adafruit_Circuit_Playground_Express-eagle-import:VREG_SOT23-5 -> 001-rescue:VREG_SOT23-5-Adafruit_Circuit_Playground_Express-eagle-import
- VCC1: renamed from VCC?; symbol Adafruit_Circuit_Playground_Express-eagle-import:SEWTAP-ALLIGATOR -> 001-rescue:SEWTAP-ALLIGATOR-Adafruit_Circuit_Playground_Express-eagle-import
- gave numbers to parts that had none: 1
Connections:
- net labels removed: 1.2V
- wire segments 335 -> 333
Other:
- moved on the sheet: C1, C7, C9

Commit message: Update Schematic SAMD21G & SPI
Parts:
- removed LED10, LED11, LED6, LED7, LED8, LED9: WS2812B3535, Adafruit Circuit Playground Express:LED3535, symbol 001-rescue:WS2812B3535-Adafruit_Circuit_Playground_Express-eagle-import
- removed R13, R14: 10k, Adafruit Circuit Playground Express:0603-NO, symbol 001-rescue:RESISTOR_0603_NOOUT-Adafruit_Circuit_Playground_Express-eagle-import
- removed R6: 10K, OSHwi:R_0805_HandSoldering, symbol 001-rescue:RESISTOR_0603_NOOUT-Adafruit_Feather_M0_Express-eagle-import
- removed TP1, TP2: TESTPOINTROUND1.5MM, Adafruit Circuit Playground Express:TESTPOINT_ROUND_1.5MM, symbol 001-rescue:TESTPOINTROUND1.5MM-Adafruit_Circuit_Playground_Express-eagle-import
- removed U$1: ATSAMD21G18MU, Adafruit Circuit Playground Express:TQFN48_7MM, symbol 001-rescue:ATSAMD21G_QFN-Adafruit_Circuit_Playground_Express-eagle-import
- removed U2: SPIFLASH_SOIC8208MIL, symbol 001-rescue:SPIFLASH_SOIC8208MIL-Adafruit_Feather_M0_Express-eagle-import
- removed U4: SPI FLASH, Adafruit Circuit Playground Express:SOIC8_150MIL, symbol 001-rescue:SPIFLASH_SOIC8-Adafruit_Circuit_Playground_Express-eagle-import
- added R?: 10K, symbol Device:R_Small
- added U?: SPI FLASH, Package_SO:SOIC-8_5.23x5.23mm_P1.27mm, symbol Memory_Flash:W25Q32JVSS
- C1, C7, C9: symbol device:C_Small -> 001-rescue:C_Small-device
- J26: symbol conn:Micro_SD_Card_Det -> 001-rescue:Micro_SD_Card_Det-conn
- TP1: renamed from J25; value TEST_1P -> TESTPOINTROUND1.5MM; symbol conn:TEST_1P -> 001-rescue:TEST_1P-conn
- TP2: renamed from J24; value TEST_1P -> TESTPOINTROUND1.5MM; symbol conn:TEST_1P -> 001-rescue:TEST_1P-conn
- U3: symbol oshwi_M0:ATSAMD21G18A-AUT -> 001-rescue:ATSAMD21G18A-AUT-oshwi_M0
- Y1: symbol device:Crystal -> 001-rescue:Crystal-device
Connections:
- net labels added: SWCLK-SPK_SD
- net labels removed: D2_FLASHMISO, D2_FLASH_MISO, D3_FLASHSCK, D3_FLASH_SCK, D4_FLASHMOSI, D4_FLASH_MOSI, D7, FLASH_CS, LIS_SCL, LIS_SDA, RXLED, SWCLK, SWCLK/SPK_SD, TXLED
- wire segments 333 -> 283
- no-connect marks 11 -> 13
Other:
- note added: "Flash Memory"
- note removed: "ATSAMD21 MICROCONTROLLER"
- note removed: "Flash Memory \nInternal SPI on SERCOM 2"
- note removed: "NeoPixels"
- note removed: "RXD"
- note removed: "SERCOM 1: internal I2C\nSERCOM 3: internal SPI\nSERCOM 4: Serial\nSERCOM 5: external I2C"
- note removed: "SPI FLASH"
- note removed: "TXD"
- note removed: "USBHOSTEN"
- moved on the sheet: 3.3VTAP1, 3V3TAP1, BATT1, C1, C11, C12, C13, C14, C15, C7, C8, C9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

Commit message: Add tft-shield project
Parts:
- removed C4, C5: 10µF, OSHwi:C_0805_HandSoldering, symbol 001-rescue:CAP_CERAMIC0805-NOOUTLINE-Adafruit_Feather_M0_Express-eagle-import
- removed C6: 1uF, OSHwi:C_0805_HandSoldering, symbol 001-rescue:CAP_CERAMIC0603_NO-Adafruit_Feather_M0_Express-eagle-import
- removed D1: MBRA120, OSHwi:D_SOD-123, symbol wickerlib:DIODE-SCHOTTKY-40V-1A-MBRA140-SMA
- removed PTC1: 500mA, symbol Adafruit_0.96in_160x80_TFT_Display-eagle-import:500mA
- removed R1, R3: 100k, OSHwi:R_0805_HandSoldering, symbol 001-rescue:RESISTOR_0603_NOOUT-Adafruit_Feather_M0_Express-eagle-import
- removed R2: 100K, OSHwi:R_0805_HandSoldering, symbol 001-rescue:RESISTOR_0603_NOOUT-Adafruit_Feather_M0_Express-eagle-import
- removed U1: AP2112-3.3, OSHwi:SOT-23-5_HandSoldering, symbol 001-rescue:VREG_SOT23-5-Adafruit_Feather_M0_Express-eagle-import
- removed U?: SPI FLASH, Package_SO:SOIC-8_5.23x5.23mm_P1.27mm, symbol Memory_Flash:W25Q32JVSS
- removed X1: microUSB, Oshwi_M0:4UCONN_20329_V2, symbol 001-rescue:USB_MICRO_20329_V2-Adafruit_Feather_M0_Express-eagle-import
- removed X2: JSTPH, Oshwi_M0:JSTPH2, symbol 001-rescue:CON_JST_PH_2PIN-Adafruit_Feather_M0_Express-eagle-import
- added C? (x3): 10uF, symbol device:C_Small
- added D?: MBRA120, Wickerlib:DIODE-SMA, symbol wickerlib:DIODE-SCHOTTKY-40V-1A-MBRA140-SMA
- added F2: 500mA, symbol device:Polyfuse_Small
- added J24: USB_MICRO, symbol oshwi_M0:USB_MICRO
- added J?: JSTPH, symbol conn:CONN_01X02
- added R2, R6: 100k, symbol device:R_Small
- added R?: 100K, symbol device:R_Small
- added U2: Memory_Flash, Package_SO:SOIC-8_5.23x5.23mm_P1.27mm, symbol oshwi_M0:Memory_Flash
- added U?: AP2127K-3.3, TO_SOT_Packages_SMD:SOT-23-5, symbol regul:AP2127K-3.3
- R1: renamed from R?; symbol Device:R_Small -> 001-rescue:R_Small-Device
Connections:
- wire segments 283 -> 287
- no-connect marks 13 -> 12
Other:
- note added: "ID"

Commit message: Add Draw settings in Docs TFT
Parts:
- J24: symbol oshwi_M0:USB_MICRO -> 001-rescue:USB_MICRO-oshwi_M0
- U2: symbol oshwi_M0:Memory_Flash -> 001-rescue:Memory_Flash-oshwi_M0
Changed lines of the file:
@@
 $EndComp
 $Comp
-L oshwi_M0:Memory_Flash U2
+L 001-rescue:Memory_Flash-oshwi_M0 U2
 U 1 1 5CEAEE20
 P 8400 3750
@@
 $EndComp
 $Comp
-L oshwi_M0:USB_MICRO J24
+L 001-rescue:USB_MICRO-oshwi_M0 J24
 U 1 1 5CF4E9B6
 P 6925 1650
