File: 2019/Oshwi_ESP32_Back_01/Oshwi_ESP32.sch (KiCad schematic (older format))
At the start: 27 parts, among them J4 JSTPH, P1 CONN_01X08, P2 CONN_01X08, Q1 S8050, SW1 SW_Push, SW3 SW_Push, U3 TFT_0.9680*160, U5 AP2112-3.3, X1 ESP32_WROOM32-32D-Gus

Commit message: Add changes to ArtWork 2019
Parts:
- removed JP1: Jumper_NO, Jumper:SolderJumper-2_P1.3mm_Open_TrianglePad1.0x1.5mm, symbol Device:Jumper_NO_Small
- added A1: ANT, Cats_ArduinoShieldLoRa:SMA_EDGELAUNCH_UFL, symbol Oshwi_ESP32-rescue:ANT-Cats_GPSLoRa-cache-wemos-01-rescue
- added C7: 1u, Capacitor_SMD:C_0805_2012Metric_Pad1.29x1.40mm_HandSolder, symbol Oshwi_ESP32-rescue:CP1_Small-Device-wemos-01-rescue
- added C8: 10u, Capacitor_SMD:C_0805_2012Metric_Pad1.29x1.40mm_HandSolder, symbol Oshwi_ESP32-rescue:CP1_Small-Device-wemos-01-rescue
- added J1: CONN_01X08, Connector_PinSocket_2.54mm:PinSocket_1x08_P2.54mm_Vertical, symbol Oshwi_ESP32-rescue:CONN_01X08-conn-001-rescue
- added J2: Conn_01x04, Connector_PinSocket_2.54mm:PinSocket_1x04_P2.54mm_WeMos, symbol Oshwi_ESP32-rescue:Conn_01x04-conn-wemos-01-rescue
- added J3: Conn_01x01, Connector_PinSocket_2.54mm:PinSocket_1x01_P2.54mm_WeMos, symbol Oshwi_ESP32-rescue:Conn_01x01-conn-wemos-01-rescue
- added JP1, JP3: HEADER-1X15, Adafruit ESP32 Huzzah Breakout:1X15_ROUND_70, symbol Oshwi_ESP32-rescue:HEADER-1X15-Adafruit_ESP32_Huzzah_Breakout-eagle-import
- added U2: AP2112-3.3, Package_TO_SOT_SMD:SOT-23-5_HandSoldering, symbol Oshwi_ESP32-rescue:VREG_SOT23-5-Adafruit_ESP32_Huzzah_Breakout-eagle-import
- added U4: RFM95W-915S2, RF_Module:HOPERF_RFM9XW_SMD_WeMos, symbol Oshwi_ESP32-rescue:RFM95W-915S2-RF_AM_FM-wemos-01-rescue
- JP2: value FTDI PORT PROG -> FTDI
- P1, P2: footprint Connector_PinHeader_2.54mm:PinHeader_1x08_P2.54mm_Vertical_SMD_Pin1Left -> D1_mini:D1_mini_Pin_Header
- U3: footprint Display:TFT_0.96_SPI -> (none)
- renumbered C4 to C?, D4 to D?, D5 to D?, SW1 to SW?
Connections:
- net labels added: +5V, A0, CS, D3, D4, D8, DC, G2, G3, G4, G5, GPIO18, GPIO2, GPIO23, GPIO4, GPIO5, RES, RST, RX, SCL, SDA, TX
- net labels removed: GPIO18_SCL, GPIO23_SDA, GPIO2_DC, GPIO4_RES, GPIO5_CS
- wire segments 103 -> 178
- no-connect marks 15 -> 7
Other:
- note added: "D1 Mini Shield"
- note added: "GPIO0"
- note added: "GPIO12"
- note added: "GPIO13"
- note added: "GPIO14"
- note added: "GPIO15"
- note added: "GPIO16"
- note added: "GPIO2"
- note added: "GPIO4"
- note added: "GPIO5"
- note removed: "+3.3V"
- note removed: "+5V"
- note removed: "A0"
- note removed: "D1 Mini LORA Shield"
- note removed: "D3"
- note removed: "D4"
- note removed: "D8"
- note removed: "DIO0"
- note removed: "DIO1"
- note removed: "GND"
- note removed: "MISO"
- note removed: "MOSI"
- note removed: "NSS"
- note removed: "RESET"
- note removed: "RX"
- note removed: "TX"
- moved on the sheet: C6, JP2, P1, P2, U3
