File: 2017/Oshpark_Version/001.sch (KiCad schematic (older format))
At the start: 39 parts, among them J1 CONN_01X02, J10 TEST_1P, J11 TEST_1P, J12 TEST_1P, J13 TEST_1P, J14 TEST_1P, J15 TEST_1P, J16 TEST_1P, J17 GS2, J2 TEST_1P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

Commit message: Continue the Design of ESP32 Badge
Parts:
- C1, C2, C3, C4: symbol CAP -> 001-rescue:CAP
- D1: symbol DIODE-SCHOTTKY-40V-1A-MBRA140-SMA -> 001-rescue:DIODE-SCHOTTKY-40V-1A-MBRA140-SMA
- D2: symbol LED -> 001-rescue:LED
- J1: symbol CONN_01X02 -> 001-rescue:CONN_01X02
- J10, J11, J12, J13, J14, J15, J16, J2, J3, J4, J5, J6, J7, J8, J9: symbol TEST_1P -> 001-rescue:TEST_1P
- J17: symbol GS2 -> 001-rescue:GS2
- LED1, LED2, LED3, LED4, LED5: symbol LED-RGB-WS2812B-4SMD -> 001-rescue:LED-RGB-WS2812B-4SMD
- R1, R2, R3, R4, R5, R6, R7: symbol R -> 001-rescue:R
- SW1, SW2: symbol SW_Push -> 001-rescue:SW_Push
- U1: symbol ESP-12 -> 001-rescue:ESP-12
- U2: symbol SPX3819M5-L-1-8-RESCUE-001 -> 001-rescue:SPX3819M5-L-1-8-RESCUE-001
Connections:
- wire segments 70 -> 84
