File: 2017/Oshpark_Version/001.kicad_pcb (KiCad board)
At the start: 2 copper layers, 74.7 x 96.8 mm, 69 parts, among them J1 CONN_01X02, J10 TEST_1P, J11 TEST_1P, J12 TEST_1P, J13 TEST_1P, J14 TEST_1P, J15 TEST_1P, J16 TEST_1P, J17 GS2, J2 TEST_1P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

Commit message: update es8266 design
Parts:
- added REF**: JST_PH_B2B-PH-SM4-TB_1x02-1MP_P2.00mm_Vertical, Connector_JST:JST_PH_B2B-PH-SM4-TB_1x02-1MP_P2.00mm_Vertical, F.Cu at (160.5, 77.3)
