File: 2019/Oshwi_ESP32/Oshwi_ESP32.sch (KiCad schematic (older format))
At the start: 27 parts, among them J4 JSTPH, P1 CONN_01X08, P2 CONN_01X08, Q1 S8050, SW1 SW_Push, SW3 SW_Push, U3 TFT_0.9680*160, U5 AP2112-3.3, X1 ESP32_WROOM32-32D-Gus

Commit message: Continue the Design of ESP32 Badge
Parts:
- removed D1: MBR120, Diode_SMD:D_SOD-123, symbol Device:D_Schottky_Small
- removed D4: 1N4148, Diode_SMD:D_SOD-323, symbol Diode:1N4148
- removed JP2: FTDI PORT PROG, Adafruit ESP32 Huzzah Breakout:1X06_ROUND_70, symbol Oshwi_ESP32-rescue:HEADER-1X670MIL-Adafruit_ESP32_Huzzah_Breakout-eagle-import
- removed P1, P2: CONN_01X08, Connector_PinHeader_2.54mm:PinHeader_1x08_P2.54mm_Vertical_SMD_Pin1Left, symbol Oshwi_ESP32-rescue:CONN_01X08-wemos-01-rescue
- removed R2: 10K, Adafruit ESP32 Huzzah Breakout:0603-NO, symbol Oshwi_ESP32-rescue:RESISTOR_0603_NOOUT-Adafruit_ESP32_Huzzah_Breakout-eagle-imp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
- removed U5: AP2112-3.3, Package_TO_SOT_SMD:SOT-23-5, symbol Regulator_Linear:AP2112K-3.3
- added CAP1: TOUCH 1, Wickerlib:CAPSENSE-CIRCLE-D10MM, symbol wickerlib:CAPSENSE_CIRCLE
- added CAP2: TOUCH 2, Wickerlib:CAPSENSE-CIRCLE-D10MM, symbol wickerlib:CAPSENSE_CIRCLE
- added D1, D4, D6, D7, D8: WS2812B, LED_SMD:LED_WS2812B_PLCC4_5.0x5.0mm_P3.2mm, symbol LED:WS2812B
- added J1: Conn_01x06, symbol Connector_Generic:Conn_01x06
- added J? (x2): Conn_01x08, symbol Connector_Generic:Conn_01x08
- added R2: 10K, Resistor_SMD:R_0805_2012Metric_Pad1.15x1.40mm_HandSolder, symbol Device:R_Small
- added U1: AP2112-3.3, Package_TO_SOT_SMD:SOT-23-5, symbol Oshwi_ESP32:AP2112K-3.3
- C3: value 10uF -> 1uF
- C5: value 10uF -> 22nF
Connections:
- net VCC is gone; now on net +3V3: JP1.1, R4.2, U3.12 (LEDA)
- net +3V3: now also R1.1, D1.1 (VDD), D4.1 (VDD), D6.1 (VDD), D7.1 (VDD), D8.1 (VDD), J?.1 (Pin_1), J?.1 (Pin_1), R2.1, U1.5 (VOUT)
- net GND: now also D1.3 (VSS), D4.3 (VSS), D6.3 (VSS), D7.3 (VSS), D8.3 (VSS), J1.6 (Pin_6), J?.2 (Pin_2), U1.2 (GND)
- net RESET: now also R2.2
- net RXD: now also J?.7 (Pin_7)
- net RXD_5V: now also J1.3 (Pin_3)
- net TXD: now also J1.2 (Pin_2), J?.8 (Pin_8)
- net VIN: now also C1.1, D2.1 (K), J1.4 (Pin_4), U1.1 (VIN), U1.3 (EN)
- net GPIO13 renamed GPIO13_SDA
- net GPIO13_SDA: now also U3.3 (SDA); no longer R1.1
- net GPIO14 renamed GPIO14_SCL
- net GPIO14_SCL: now also U3.4 (SCL)
- net GPIO15 renamed GPIO15_CS
- net GPIO15_CS: now also U3.7 (CS)
- net GPIO16 renamed GPIO16_RES
- net GPIO16_RES: now also J?.8 (Pin_8)
- net GPIO17 renamed GPIO17_D0
- net GPIO17_D0: now also J?.6 (Pin_6)
- net GPIO18_SCL renamed GPIO18_SCK
- net GPIO18_SCK: now also J?.5 (Pin_5); no longer U3.4 (SCL)
- net GPIO19 renamed GPIO19_MISO
- net GPIO19_MISO: now also J?.4 (Pin_4)
- net GPIO21 renamed GPIO21_DIO1
- net GPIO21_DIO1: now also J?.5 (Pin_5)
- net GPIO22 renamed GPIO22_DIO0
- net GPIO22_DIO0: now also J?.6 (Pin_6)
- net GPIO23_SDA renamed GPIO23_MOSI
- net GPIO23_MOSI: now also J?.3 (Pin_3); no longer U3.3 (SDA)
- net GPIO25 renamed GPIO25_D3
- net GPIO25_D3: now also J?.4 (Pin_4)
- net GPIO26 renamed GPIO26_D4
- net GPIO26_D4: now also J?.3 (Pin_3)
- net GPIO27 renamed GPIO27_TOUCH
- net GPIO27_TOUCH: now also CAP2.1 (BUTTON)
- net GPIO2_DC renamed GPIO2_NEOPIXEL
- net GPIO2_NEOPIXEL: now also D1.4 (DIN); no longer U3.5 (RS)
- net GPIO32 renamed GPIO32_RES
- net GPIO32_RES: now also U3.6 (RES)
- net GPIO33 renamed GPIO33_DC
- net GPIO33_DC: now also U3.5 (RS)
- net GPIO36 renamed GPIO36_A0
- net GPIO36_A0: now also J?.7 (Pin_7)
- net GPIO4_RES renamed GPIO4_TOUCH
- net GPIO4_TOUCH: now also CAP1.1 (BUTTON); no longer U3.6 (RES)
- net GPIO5_CS renamed GPIO5_NSS
- net GPIO5_NSS: now also J?.2 (Pin_2); no longer U3.7 (CS)
- new net: D1.2 (DOUT), D4.4 (DIN)
- new net: D4.2 (DOUT), D6.4 (DIN)
- new net: D6.2 (DOUT), D7.4 (DIN)
- new net: D7.2 (DOUT), D8.4 (DIN)
Other:
- note added: "D0"
- note added: "D5_SCK"
- note added: "D6_MISO"
- note added: "D7_MOSI"
- note added: "D8_CS_NSS"
- note added: "ESP32"
- note added: "LCD TFT"
- note added: "LORA Shield Port"
- note added: "Mini"
- note added: "Neopixels"
- note added: "On"
- note added: "Power & Filtering"
- note added: "RES"
- note added: "SCL"
- note added: "SDA"
- note added: "Touch Pads"
- note added: "VDD +\nVSS -"
- note removed: "+5V"
- note removed: "D1 Mini LORA Shield"
- note removed: "D8"
- note removed: "MISO"
- note removed: "MOSI"
- note removed: "NSS"
- note removed: "RESET"
- moved on the sheet: C1, C2, C3, C4, D2, D5, J4, SW1, SW3

Commit message: update es8266 design
Parts:
- removed D7, D8: WS2812B, LED_SMD:LED_WS2812B_PLCC4_5.0x5.0mm_P3.2mm, symbol LED:WS2812B
- removed X1: ESP32_WROOM32-32D-Gus, symbol RF_Module:ESP32_WROOM32-32D-Gus
- added D3, D5: WS2812B, Oshwi_ESP32:WS2812B, symbol LED:WS2812B
- added U3: ESP32-WROOM-32D, RF_Module:ESP32-WROOM-32, symbol RF_Module:ESP32-WROOM-32D
- added U4: Oshwi_Edge_Cut, Oshwi_ESP32:Oshwi_ESP32, symbol Oshwi_ESP32:Oshwi_Edge_Cut
- C1, C2, C3, C5: footprint (none) -> Capacitor_SMD:C_0805_2012Metric_Pad1.15x1.40mm_HandSolder
- CAP1: footprint Wickerlib:CAPSENSE-CIRCLE-D10MM -> Oshwi_ESP32:Touch_1
- CAP2: footprint Wickerlib:CAPSENSE-CIRCLE-D10MM -> Oshwi_ESP32:Touch_2
- D2: renamed from D1; footprint LED_SMD:LED_WS2812B_PLCC4_5.0x5.0mm_P3.2mm -> Oshwi_ESP32:WS2812B
- D4, D6: footprint LED_SMD:LED_WS2812B_PLCC4_5.0x5.0mm_P3.2mm -> Oshwi_ESP32:WS2812B
- D8: renamed from D3; footprint (none) -> LED_SMD:LED_0805_2012Metric_Pad1.15x1.40mm_HandSolder
- J1: renamed from J?; value Conn_01x08 -> RES-A0; footprint (none) -> Connector_PinSocket_2.54mm:PinSocket_1x08_P2.54mm_Vertical_SMD_Pin1Left
- J2: renamed from J?; value Conn_01x08 -> TXD-RXD; footprint (none) -> Connector_PinSocket_2.54mm:PinSocket_1x08_P2.54mm_Vertical_SMD_Pin1Left
- J3: renamed from J1; footprint (none) -> Connector_PinSocket_2.54mm:PinSocket_1x06_P2.54mm_Vertical_SMD_Pin1Left
- J4: footprint Connector_JST:JST_PH_B2B-PH-SM4-TB_1x02-1MP_P2.00mm_Vertical -> Oshwi_ESP32:JSTPH2
- SW1: renamed from SW3; footprint (none) -> Oshwi_ESP32:SW_SPST_B3U-1000P
- SW2: renamed from SW1; footprint (none) -> Oshwi_ESP32:SW_SPST_B3U-1000P
- renumbered C6 to C4, C4 to C6, D2 to D1, D5 to D7, R5 to R1, R3 to R2, R4 to R3, R2 to R4, R1 to R5, U3 to U2
Connections:
- net +3V3: now also D3.1 (VDD), D5.1 (VDD), U3.2 (VDD)
- net GND: now also D3.3 (VSS), D5.3 (VSS), U3.1 (GND), U3.15 (GND), U3.38 (GND); no longer C6.2, SW2.1
- net GPI34: now also U3.6 (IO34)
- net GPI35: now also U3.7 (IO35)
- net GPIO0: now also U3.25 (IO0)
- net GPIO12: now also U3.14 (IO12)
- net GPIO13_SDA: now also U3.16 (IO13)
- net GPIO14_SCL: now also U3.13 (IO14)
- net GPIO15_CS: now also U3.23 (IO15)
- net GPIO16_RES: now also U3.27 (IO16)
- net GPIO17_D0: now also U3.28 (IO17)
- net GPIO18_SCK: now also U3.30 (IO18)
- net GPIO19_MISO: now also U3.31 (IO19)
- net GPIO21_DIO1: now also U3.33 (IO21)
- net GPIO22_DIO0: now also U3.36 (IO22)
- net GPIO23_MOSI: now also U3.37 (IO23)
- net GPIO25_D3: now also U3.10 (IO25)
- net GPIO26_D4: now also U3.11 (IO26)
- net GPIO27_TOUCH: now also U3.12 (IO27)
- net GPIO2_NEOPIXEL: now also U3.24 (IO2)
- net GPIO32_RES: now also U3.8 (IO32)
- net GPIO33_DC: now also U3.9 (IO33)
- net GPIO36_A0: now also U3.4 (SENSOR_VP)
- net GPIO39: now also U3.5 (SENSOR_VN)
- net GPIO4_TOUCH: now also U3.26 (IO4)
- net GPIO5_NSS: now also U3.29 (IO5)
- net RESET: now also U3.3 (EN)
- net RXD: now also U3.34 (RXD0/IO3)
- net TXD: now also U3.35 (TXD0/IO1)
- net at D4.4 (DIN): now also D3.2 (DOUT); no longer D2.2 (DOUT)
- net at D4.2 (DOUT): now also D5.4 (DIN); no longer D6.4 (DIN)
- new net: C6.2, SW2.1
- new net: D2.2 (DOUT), D3.4 (DIN)
- new net: D5.2 (DOUT), D6.4 (DIN)
- no-connect marks 15 -> 17
Other:
- note added: "SDI"
- note removed: "SHI"
- moved on the sheet: C5, D2, J1, J2
